File: KiCAD/AudioAmpEEL/AudioAmpEEL.kicad_pcb (KiCad board)
At the start: 2 copper layers, 81.5 x 44 mm, 23 parts, among them J1 Signal In (10mV), J2 Amplified Output, J3 -9V GND +9V, Q1 2N3904, Q2 2N3904, Q3 2N3906

Commit message: Quick Fix for PCB
Routing:
- net /Vee (-9V): track 76.3 -> 115.4 mm
- net Net-(Q1-C): track 19.2 -> 16.5 mm
- net Net-(D1-A): track 25.5 -> 23.2 mm
- net /Vout: track 33.9 -> 31.6 mm
- net Net-(Q1-E): track 19.1 -> 17.4 mm
- net Net-(D2-K): track 26.0 -> 24.8 mm
Changed lines of the file:
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@@
       (outputformat 1)
       (mirror false)
-      (drillshape 1)
+      (drillshape 0)
       (scaleselection 1)
-      (outputdirectory "")
+      (outputdirectory "GerberFiles/")
     )
   )
@@
   (segment (start 124 92) (end 124 86.08) (width 0.2) (layer "B.Cu") (net 2))
   (segment (start 132 93) (end 124 93) (width 0.2) (layer "B.Cu") (net 2))
-  (segment (start 132 86.08) (end 137.58 86.08) (width 0.2) (layer "B.Cu") (net 3))
-  (segment (start 140 88.5) (end 140 93) (width 0.2) (layer "B.Cu") (net 3))
-  (segment (start 137.58 86.08) (end 140 88.5) (width 0.2) (layer "B.Cu") (net 3))
+  (segment (start 138.92 93) (end 132 86.08) (width 0.2) (layer "B.Cu") (net 3))
   (segment (start 132 91.73) (end 132 86.08) (width 0.2) (layer "B.Cu") (net 3))
+  (segment (start 140 93) (end 138.92 93) (width 0.2) (layer "B.Cu") (net 3))
   (segment (start 149 93) (end 142 93) (width 0.2) (layer "B.Cu") (net 4))
   (segment (start 149 93) (end 149 100.42) (width 0.2) (layer "B.Cu") (net 4))
   (segment (start 151.5 93) (end 149 93) (width 0.2) (layer "B.Cu") (net 4))
   (segment (start 149 86.58) (end 149 93) (width 0.2) (layer "B.Cu") (net 4))
-  (segment (start 141 102) (end 140 101) (width 0.2) (layer "B.Cu") (net 5))
-  (segment (start 140 101) (end 132 101) (width 0.2) (layer "B.Cu") (net 5))
-  (segment (start 141 105) (end 141 102) (width 0.2) (layer "B.Cu") (net 5))
+  (segment (start 141 105) (end 136 105) (width 0.2) (layer "B.Cu") (net 5))
+  (segment (start 136 105) (end 132 101) (width 0.2) (layer "B.Cu") (net 5))
   (segment (start 132 94.27) (end 132 101) (width 0.2) (layer "B.Cu") (net 5))
-  (segment (start 159 109.5) (end 158 110.5) (width 0.2) (layer "B.Cu") (net 6))
   (segment (start 141 107.5) (end 146 112.5) (width 0.2) (layer "B.Cu") (net 6))
+  (segment (start 109 89) (end 106.5 91.5) (width 0.2) (layer "B.Cu") (net 6))
   (segment (start 137.34 111.16) (end 141 107.5) (width 0.2) (layer "B.Cu") (net 6))
+  (segment (start 173.21 105) (end 163.5 105) (width 0.2) (layer "B.Cu") (net 6))
+  (segment (start 106.5 108.5) (end 109 111) (width 0.2) (layer "B.Cu") (net 6))
+  (segment (start 156 110.5) (end 158 110.5) (width 0.2) (layer "B.Cu") (net 6))
   (segment (start 109.16 111.16) (end 109 111) (width 0.2) (layer "B.Cu") (net 6))
   (segment (start 124 111.16) (end 109.16 111.16) (width 0.2) (layer "B.Cu") (net 6))
-  (segment (start 163.5 105) (end 159.5 105) (width 0.2) (layer "B.Cu") (net 6))
-  (segment (start 158 110.5) (end 156 110.5) (width 0.2) (layer "B.Cu") (net 6))
+  (segment (start 178.64 110.43) (end 173.21 105) (width 0.2) (layer "B.Cu") (net 6))
   (segment (start 178.65 99.26) (end 180.5 101.11) (width 0.2) (layer "B.Cu") (net 6))
   (segment (start 180.5 108.57) (end 178.64 110.43) (width 0.2) (layer "B.Cu") (net 6))
+  (segment (start 106.5 91.5) (end 106.5 108.5) (width 0.2) (layer "B.Cu") (net 6))
   (segment (start 146 112.5) (end 154 112.5) (width 0.2) (layer "B.Cu") (net 6))
   (segment (start 132 111.16) (end 137.34 111.16) (width 0.2) (layer "B.Cu") (net 6))
   (segment (start 154 112.5) (end 156 110.5) (width 0.2) (layer "B.Cu") (net 6))
+  (segment (start 158 110.5) (end 163.5 105) (width 0.2) (layer "B.Cu") (net 6))
   (segment (start 180.5 101.11) (end 180.5 108.57) (width 0.2) (layer "B.Cu") (net 6))
-  (segment (start 159 105.5) (end 159 109.5) (width 0.2) (layer "B.Cu") (net 6))
   (segment (start 124 111.16) (end 132 111.16) (width 0.2) (layer "B.Cu") (net 6))
-  (segment (start 159.5 105) (end 159 105.5) (width 0.2) (layer "B.Cu") (net 6))
   (segment (start 159.62 79.96) (end 156 76.34) (width 0.2) (layer "B.Cu") (net 8))
   (segment (start 147 74.5) (end 154.16 74.5) (width 0.2) (layer "B.Cu") (net 8))
@@
   (segment (start 110 76) (end 117 76) (width 0.2) (layer "B.Cu") (net 8))
   (segment (start 161.27 81.23) (end 156 86.5) (width 0.2) (layer "B.Cu") (net 9))
-  (segment (start 150.92 76.42) (end 149 76.42) (width 0.2) (layer "B.Cu") (net 9))
-  (segment (start 152.5 78) (end 150.92 76.42) (width 0.2) (layer "B.Cu") (net 9))
   (segment (start 164 81.23) (end 161.27 81.23) (width 0.2) (layer "B.Cu") (net 9))
-  (segment (start 152.5 85) (end 152.5 78) (width 0.2) (layer "B.Cu") (net 9))
-  (segment (start 156 86.5) (end 154 86.5) (width 0.2) (layer "B.Cu") (net 9))
-  (segment (start 154 86.5) (end 152.5 85) (width 0.2) (layer "B.Cu") (net 9))
-  (segment (start 159 101) (end 159 103) (width 0.2) (layer "B.Cu") (net 10))
+  (segment (start 149 79.5) (end 156 86.5) (width 0.2) (layer "B.Cu") (net 9))
+  (segment (start 149 76.42) (end 149 79.5) (width 0.2) (layer "B.Cu") (net 9))
   (segment (start 152.5 109.5) (end 152.5 101.5) (width 0.2) (layer "B.Cu") (net 10))
-  (segment (start 159.73 103.73) (end 163.5 103.73) (width 0.2) (layer "B.Cu") (net 10))
-  (segment (start 158.34 100.34) (end 159 101) (width 0.2) (layer "B.Cu") (net 10))
+  (segment (start 156 100.34) (end 159.39 103.73) (width 0.2) (layer "B.Cu") (net 10))
   (segment (start 152.5 101.5) (end 153.66 100.34) (width 0.2) (layer "B.Cu") (net 10))
   (segment (start 153.66 100.34) (end 156 100.34) (width 0.2) (layer "B.Cu") (net 10))
-  (segment (start 156 100.34) (end 158.34 100.34) (width 0.2) (layer "B.Cu") (net 10))
-  (segment (start 159 103) (end 159.73 103.73) (width 0.2) (layer "B.Cu") (net 10))
   (segment (start 149 110.58) (end 151.42 110.58) (width 0.2) (layer "B.Cu") (net 10))
+  (segment (start 159.39 103.73) (end 163.5 103.73) (width 0.2) (layer "B.Cu") (net 10))
   (segment (start 151.42 110.58) (end 152.5 109.5) (width 0.2) (layer "B.Cu") (net 10))
-  (segment (start 170 92.42) (end 173.92 92.42) (width 0.2) (layer "B.Cu") (net 11))
-  (segment (start 175 100) (end 178.64 103.64) (width 0.2) (layer "B.Cu") (net 11))
-  (segment (start 175 93.5) (end 175 100) (width 0.2) (layer "B.Cu") (net 11))
+  (segment (start 170 92.42) (end 170 99.25) (width 0.2) (layer "B.Cu") (net 11))
+  (segment (start 170 99.25) (end 178.64 107.89) (width 0.2) (layer "B.Cu") (net 11))
   (segment (start 170 89.08) (end 178.63 89.08) (width 0.2) (layer "B.Cu") (net 11))
   (segment (start 178.63 89.08) (end 178.65 89.1) (width 0.2) (layer "B.Cu") (net 11))
-  (segment (start 178.64 103.64) (end 178.64 107.89) (width 0.2) (layer "B.Cu") (net 11))
   (segment (start 170 93) (end 170 89.08) (width 0.2) (layer "B.Cu") (net 11))
-  (segment (start 173.92 92.42) (end 175 93.5) (width 0.2) (layer "B.Cu") (net 11))
   (segment (start 166.42 82.5) (end 164 82.5) (width 0.2) (layer "B.Cu") (net 12))
   (segment (start 170 78.92) (end 166.42 82.5) (width 0.2) (layer "B.Cu") (net 12))

Commit message: Update PCB & Gerber Files
Parts:
- J1: value Signal In (10mV) -> 10kHz
- moved RLoad1 1.83 mm to (178.5, 101.1)
Routing:
- net /Vout: track 31.6 -> 37.4 mm
- net Net-(D2-K): track 24.8 -> 22.0 mm
- net /Vcc (+9V): track 62.7 -> 60.1 mm
- net /Vee (-9V): track 115.4 -> 113.7 mm
- net /Vin: track 12.4 -> 10.6 mm
Other:
- board text added: "+OUT"
- board text added: "-OUT"
- board text added: "10mV in"
- board text added: "Dual Supply Single Channel Audio Amplifier: fc = 10kHz"
- board text added: "GND"
- board text added: "Joel Brigida: EEL-3118L"
- board text removed: "Joel Brigida Audio Amplifier"
