File: KiCAD/AudioAmpEELv2/AudioAmpEELv2.kicad_pcb (KiCad board)
At the start: 2 copper layers, 81.5 x 44 mm, 25 parts, among them J1 Signal In (10mV), J2 Amplified Output, J3 -9V GND +9V, Q1 2N3904, Q2 2N3904, Q3 2N3906

Commit message: Update Gerber Files & PCB Layout
Parts:
- moved Rc1 3.58 mm to (129.0, 84.2)
- moved R4a1 3.50 mm to (152.5, 110.6)
- moved D2 3.00 mm to (146.0, 110.6)
- moved Q1 3.00 mm to (129.0, 94.3)
- moved R4b1 3.00 mm to (159.5, 110.7)
- moved Re1 3.00 mm to (129.0, 111.2)
- moved C2 2.96 mm to (137.0, 93.0)
- moved C3 2.96 mm to (138.0, 105.0)
- moved R1 2.77 mm to (122.0, 84.2)
- moved Q3 2.64 mm to (165.5, 106.2)
- moved C4 2.49 mm to (115.5, 79.0)
- moved C1 2.46 mm to (115.5, 93.0)
- moved R3a1 2.39 mm to (152.5, 84.1)
- moved R2 2.00 mm to (122.0, 111.2)
- moved R3b1 1.05 mm to (159.4, 85.5)
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Routing:
- net Net-(Q1-C): track 16.5 -> 19.8 mm
- net Net-(D1-A): track 31.5 -> 28.3 mm
- net /Vee (-9V): track 110.1 -> 113.3 mm
- net Net-(Q3-E): track 5.66 -> 8.29 mm
- net Net-(D1-K): track 24.6 -> 27.1 mm
- net /Vin: track 10.6 -> 8.19 mm
- net Net-(R3a1-Pad1): track 13.0 -> 11.6 mm
- net Net-(Q1-B): track 26.9 -> 28.3 mm
- net /Vcc (+9V): track 63.5 -> 64.3 mm
Other:
- board text added: "K"
